Commit message: Update: add shivam's code

File: source/robot_lab/data/Robots/go2_with_airbot/urdf/go2_with_airbot_vis_flip.urdf (robot description, URDF)
Before this commit: robot go2_with_arm, 43 links, 42 joints
Joints:
- joint airbot_j1: type fixed -> revolute
- joint airbot_j2: type fixed -> revolute
- joint airbot_j3: type fixed -> revolute
- joint airbot_j4: type fixed -> revolute
- joint airbot_j5: type fixed -> revolute
- joint airbot_j6: type fixed -> revolute
